Commit message: added gps sensor

File: vanir_description/urdf/gazebo_control.xacro (robot description, xacro)
@@ -123,3 +123,11 @@
 </sensor>
 </gazebo>
+<gazebo reference="gps_link">
+  <sensor name="navsat" type="navsat">
+    <always_on>1</always_on>
+    <update_rate>5</update_rate>
+    <topic>/gps/fix</topic>
+    <gz_frame_id>gps_link</gz_frame_id>
+  </sensor>
+</gazebo>
 </robot>

File: vanir_description/urdf/robot_core.xacro (robot description, xacro)
@@ -196,3 +196,11 @@
   <material>Gazebo/Gray</material>
 </gazebo>
+<!-- GPS Sensor -->
+<link name="gps_link">
+</link>
+<joint name="gps_joint" type="fixed">
+  <parent link="base_link"/>
+  <child link="gps_link"/>
+  <origin xyz="-0.05 0 0.05" rpy="0 0 0"/>
+</joint>
 </robot>

Commit message: added imu and fixed gps plpugin

File: vanir_description/urdf/gazebo_control.xacro (robot description, xacro)
@@ -131,3 +131,12 @@
   </sensor>
 </gazebo>
+<!-- IMU  -->
+<gazebo reference="imu_link">
+  <sensor name="imu_sensor" type="imu">
+    <always_on>true</always_on>
+    <update_rate>100</update_rate>
+    <visualize>true</visualize>
+    <topic>imu</topic>
+  </sensor>
+</gazebo>
 </robot>

File: vanir_description/urdf/robot_core.xacro (robot description, xacro)
@@ -204,3 +204,12 @@
   <origin xyz="-0.05 0 0.05" rpy="0 0 0"/>
 </joint>
+<!-- IMU  -->
+<link name="imu_link">
+</link>
+<joint name="imu_joint" type="fixed">
+  <origin xyz="0 0.0 0.2" rpy="0 0 0"/>
+  <parent link="base_link"/>
+  <child link="imu_link"/>
+  <axis xyz="0 0 0" />
+</joint>
 </robot>
